File: kicad/k1-aioc/k1-aioc.kicad_pcb (KiCad board)
At the start: 2 copper layers, 21 x 31.5 mm, 47 parts, among them J1 12401832E402A, J2 Conn_01x07_Male, Q1 BC847BS, U1 MIC5330-SSYML, U2 STM32F373CBTx, Y1 8MHz/20pF

Commit message: k1-aioc Rev 1.1 with PTT2 GPIO input capabilities
Parts:
- added R18: 220R, Resistor_SMD:R_0603_1608Metric, F.Cu at (118.0, 104.8)
- added R19: 220R, Resistor_SMD:R_0603_1608Metric, F.Cu at (118.0, 103.2)
- moved R17 2.75 mm to (122.5, 103.5)
- moved C12 2.30 mm to (123.2, 101.2), turned to 90 degrees
- moved R4 1.25 mm to (121.8, 101.2), turned to -90 degrees
- moved R2 0.90 mm to (120.2, 102.8), turned to 90 degrees
- moved C13 0.75 mm to (119.5, 107.0)
- moved C9 0.75 mm to (113.5, 107.0)
- moved R10 0.75 mm to (115.0, 107.0)
- moved R11 0.75 mm to (116.5, 107.0)
- moved R12 0.75 mm to (118.0, 107.0)
- moved Q1 0.40 mm to (115.8, 109.9)
- moved R13 0.40 mm to (118.0, 109.9)
- moved C7 0.30 mm to (119.5, 100.5)
Connections:
- U2 pad 42: unconnected-(U2-Pad42) -> /PTT1-IN
- U2 pad 43: unconnected-(U2-Pad43) -> /PTT2-IN
Routing:
- net /PTT2-IN: track 0.00 -> 11.2 mm, vias 0 -> 2
- net /PTT1-IN: track 0.00 -> 10.5 mm
- net +3.3VA: track 30.8 -> 37.0 mm
- net +3V3: track 51.0 -> 54.9 mm, vias 5 -> 9
- net /RADIO-TX: track 24.2 -> 27.4 mm
- net Net-(C12-Pad1): track 7.03 -> 9.64 mm
- net /DAC_ATTEN: track 3.07 -> 5.38 mm
- net GND: track 9.36 -> 11.5 mm, vias 62 -> 57
- net /RADIO-VP-PTT2: track 4.77 -> 6.87 mm
- net /RADIO-RX-PTT1: track 30.0 -> 31.7 mm, vias 2 -> 3
- net /AFOUT: track 2.26 -> 3.51 mm
- net /RADIO-MIC: track 2.93 -> 2.18 mm
- net /PTT2: track 2.22 -> 2.97 mm
- net Net-(Q1-Pad5): track 3.15 -> 2.48 mm
- net Net-(Q1-Pad2): track 3.17 -> 2.50 mm
Other:
- board text added: "AIOC V1.1"
- board text removed: "AIOC V1.0"

Commit message: Changed PTT1 and RADIO-RX to a split-pad that is automatically connected, when a TRS connector is used. If not, then both pads can be used separately
Parts:
- R17: value N.M. -> 220R
Connections:
- net /RADIO-VP-PTT2 renamed /RADIO-PTT2
- R13 pad 1: /RADIO-RX-PTT1 -> /RADIO-PTT1
- R19 pad 1: /RADIO-RX-PTT1 -> /RADIO-PTT1
- R8 pad 1: /RADIO-RX-PTT1 -> /RADIO-RX
Routing:
- net /RADIO-RX-PTT1: track 31.7 -> 0.00 mm, vias 3 -> 0
- net /RADIO-RX: track 0.00 -> 25.3 mm, vias 0 -> 1
- net /RADIO-PTT1: track 0.00 -> 14.2 mm, vias 0 -> 2
- added copper zone on B.Cu, net /RADIO-PTT1
- added copper zone on B.Cu, net /RADIO-RX
- removed copper zone on B.Cu, net /RADIO-RX-PTT1
Changed lines of the file:
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@@
   (net 43 "/RADIO-SPK")
   (net 44 "/AFOUT")
-  (net 45 "/RADIO-RX-PTT1")
+  (net 45 "/RADIO-RX")
   (net 46 "/RADIO-TX")
-  (net 47 "/RADIO-VP-PTT2")
+  (net 47 "/RADIO-PTT2")
   (net 48 "/NRST")
   (net 49 "/SWO")
@@
   (net 59 "/DAC_ATTEN")
   (net 60 "/PTT2-IN")
+  (net 61 "/RADIO-PTT1")
   (footprint "Resistor_SMD:R_0603_1608Metric" (layer "F.Cu")
     (at 120.25 102.75 90)
@@
     (fp_line (start -0.8 0.4125) (end -0.8 -0.4125) (layer "F.Fab") (width 0.1))
     (pad "1" smd roundrect (at -0.825 0 180) (size 0.8 0.95) (layers "F.Cu" "F.Paste" "F.Mask") (roundrect_rratio 0.25)
-      (net 45 "/RADIO-RX-PTT1") (pintype "passive"))
+      (net 61 "/RADIO-PTT1") (pintype "passive"))
     (pad "2" smd roundrect (at 0.825 0 180) (size 0.8 0.95) (layers "F.Cu" "F.Paste" "F.Mask") (roundrect_rratio 0.25)
       (net 11 "/PTT1-IN") (pintype "passive"))
@@
     (fp_line (start -0.8 -0.4125) (end 0.8 -0.4125) (layer "F.Fab") (width 0.1))
     (pad "1" smd roundrect (at -0.825 0 180) (size 0.8 0.95) (layers "F.Cu" "F.Paste" "F.Mask") (roundrect_rratio 0.25)
-      (net 47 "/RADIO-VP-PTT2") (pintype "passive"))
+      (net 47 "/RADIO-PTT2") (pintype "passive"))
     (pad "2" smd roundrect (at 0.825 0 180) (size 0.8 0.95) (layers "F.Cu" "F.Paste" "F.Mask") (roundrect_rratio 0.25)
       (net 60 "/PTT2-IN") (pintype "passive"))
@@
     (fp_line (start 0.8 -0.4125) (end 0.8 0.4125) (layer "F.Fab") (width 0.1))
     (pad "1" smd roundrect (at -0.825 0 270) (size 0.8 0.95) (layers "F.Cu" "F.Paste" "F.Mask") (roundrect_rratio 0.25)
-      (net 45 "/RADIO-RX-PTT1") (pintype "passive"))
+      (net 61 "/RADIO-PTT1") (pintype "passive"))
     (pad "2" smd roundrect (at 0.825 0 270) (size 0.8 0.95) (layers "F.Cu" "F.Paste" "F.Mask") (roundrect_rratio 0.25)
       (net 36 "Net-(Q1-Pad3)") (pintype "passive"))
@@
     (fp_line (start 0.8 0.4125) (end -0.8 0.4125) (layer "F.Fab") (width 0.1))
     (pad "1" smd roundrect (at -0.825 0 270) (size 0.8 0.95) (layers "F.Cu" "F.Paste" "F.Mask") (roundrect_rratio 0.25)
-      (net 45 "/RADIO-RX-PTT1") (pintype "passive"))
+      (net 45 "/RADIO-RX") (pintype "passive"))
     (pad "2" smd roundrect (at 0.825 0 270) (size 0.8 0.95) (layers "F.Cu" "F.Paste" "F.Mask") (roundrect_rratio 0.25)
       (net 38 "/USART-TX") (pintype "passive"))
@@
       (effects (font (size 1 1) (thickness 0.15)))
     )
-    (fp_text value "N.M." (at 0 1.43) (layer "F.Fab")
+    (fp_text value "220R" (at 0 1.43) (layer "F.Fab")
       (effects (font (size 1 1) (thickness 0.15)))
     )
@@
     (fp_line (start -0.8 -0.4125) (end 0.8 -0.4125) (layer "F.Fab") (width 0.1))
     (pad "1" smd roundrect (at -0.825 0 270) (size 0.8 0.95) (layers "F.Cu" "F.Paste" "F.Mask") (roundrect_rratio 0.25)
-      (net 47 "/RADIO-VP-PTT2") (pintype "passive"))
+      (net 47 "/RADIO-PTT2") (pintype "passive"))
     (pad "2" smd roundrect (at 0.825 0 270) (size 0.8 0.95) (layers "F.Cu" "F.Paste" "F.Mask") (roundrect_rratio 0.25)
       (net 37 "Net-(Q1-Pad6)") (pintype "passive"))
@@
   (segment (start 119.011829 89.364195) (end 118.764341 89.364195) (width 0.25) (layer "F.Cu") (net 45))
   (segment (start 117.216682 89.5) (end 116.466682 90.25) (width 0.25) (layer "F.Cu") (net 45))
-  (segment (start 118.825 103.25) (end 118.25 103.25) (width 0.25) (layer "F.Cu") (net 45))
-  (segment (start 118 103.5) (end 118 104) (width 0.25) (layer "F.Cu") (net 45))
-  (segment (start 119 110.75) (end 119 109.5) (width 0.25) (layer "F.Cu") (net 45))
-  (segment (start 119 109.5) (end 118.575 109.075) (width 0.25) (layer "F.Cu") (net 45))
   (segment (start 116.466682 90.25) (end 115.116116 90.25) (width 0.25) (layer "F.Cu") (net 45))
-  (segment (start 118.575 109.075) (end 118 109.075) (width 0.25) (layer "F.Cu") (net 45))
-  (segment (start 118.25 103.25) (end 118 103.5) (width 0.25) (layer "F.Cu") (net 45))
   (segment (start 114.75 90.616116) (end 114.75 91.0875) (width 0.25) (layer "F.Cu") (net 45))
   (segment (start 118.764341 89.364195) (end 118.628536 89.5) (width 0.25) (layer "F.Cu") (net 45))
-  (via (at 118 104) (size 0.6) (drill 0.3) (layers "F.Cu" "B.Cu") (net 45))
-  (via (at 119 110.75) (size 0.6) (drill 0.3) (layers "F.Cu" "B.Cu") (net 45))
   (via (at 119.011829 89.364195) (size 0.6) (drill 0.3) (layers "F.Cu" "B.Cu") (net 45))
   (segment (start 124 92.363604) (end 123.386396 91.75) (width 0.25) (layer "B.Cu") (net 45))
-  (segment (start 118 104) (end 118 104.75) (width 0.25) (layer "B.Cu") (net 45))
   (segment (start 121.397634 91.75) (end 119.011829 89.364195) (width 0.25) (layer "B.Cu") (net 45))
   (segment (start 124 103.75) (end 124 92.363604) (width 0.25) (layer "B.Cu") (net 45))
@@
   (segment (start 124 104.5) (end 123.5 105) (width 0.25) (layer "B.Cu") (net 45))
   (segment (start 124 103.75) (end 124 104.5) (width 0.25) (layer "B.Cu") (net 45))
-  (segment (start 119 110.75) (end 119 109) (width 0.25) (layer "B.Cu") (net 45))
   (segment (start 117.030286 89.05) (end 118.44214 89.05) (width 0.25) (layer "F.Cu") (net 46))
   (segment (start 113.5 90.25) (end 114.47972 90.25) (width 0.25) (layer "F.Cu") (net 46))
@@
   (segment (start 116.168768 103.551946) (end 116.151946 103.551946) (width 0.25) (layer "B.Cu") (net 60))
   (segment (start 116.151946 103.551946) (end 114.75 102.15) (width 0.25) (layer "B.Cu") (net 60))
+  (segment (start 118.825 103.25) (end 118.25 103.25) (width 0.25) (layer "F.Cu") (net 61))
+  (segment (start 118 103.5) (end 118 104) (width 0.25) (layer "F.Cu") (net 61))
+  (segment (start 119 110.75) (end 119 109.5) (width 0.25) (layer "F.Cu") (net 61))
+  (segment (start 119 109.5) (end 118.575 109.075) (width 0.25) (layer "F.Cu") (net 61))
+  (segment (start 118.575 109.075) (end 118 109.075) (width 0.25) (layer "F.Cu") (net 61))
+  (segment (start 118.25 103.25) (end 118 103.5) (width 0.25) (layer "F.Cu") (net 61))
+  (via (at 118 104) (size 0.6) (drill 0.3) (layers "F.Cu" "B.Cu") (net 61))
+  (via (at 119 110.75) (size 0.6) (drill 0.3) (layers "F.Cu" "B.Cu") (net 61))
+  (segment (start 117.625 110.75) (end 117.05 110.175) (width 0.25) (layer "B.Cu") (net 61))
+  (segment (start 119 110.75) (end 117.625 110.75) (width 0.25) (layer "B.Cu") (net 61))
+  (segment (start 117.05 110.175) (end 117.05 104.35) (width 0.25) (layer "B.Cu") (net 61))
+  (segment (start 117.05 104.35) (end 117.4 104) (width 0.25) (layer "B.Cu") (net 61))
+  (segment (start 117.4 104) (end 118 104) (width 0.25) (layer "B.Cu") (net 61))
+  (segment (start 119 110.75) (end 119 109.5) (width 0.25) (layer "B.Cu") (net 61))
   (zone (net 1) (net_name "GND") (layer "F.Cu") (hatch edge 0.508)
     (priority 3)
@@
     )
   )
-  (zone (net 47) (net_name "/RADIO-VP-PTT2") (layer "F.Cu") (hatch edge 0.508)
+  (zone (net 47) (net_name "/RADIO-PTT2") (layer "F.Cu") (hatch edge 0.508)
     (priority 5)
     (connect_pads (clearance 0.254))
@@
     )
   )
+  (zone (net 45) (net_name "/RADIO-RX") (layer "B.Cu") (hatch edge 0.508)
+    (priority 10)
+    (connect_pads (clearance 0.254))
+    (min_thickness 0.254) (filled_areas_thickness no)
+    (fill yes (thermal_gap 0.508) (thermal_bridge_width 0.508) (smoothing fillet) (radius 0.25) (island_removal_mode 1) (island_area_min 0))
+    (polygon
+      (pts
+        (xy 123 107)
+        (xy 117.5 107)
+        (xy 117.5 104.5)
+        (xy 123 104.5)
+      )
+    )
+  )
   (zone (net 1) (net_name "GND") (layer "B.Cu") (hatch edge 0.508)
     (priority 5)
@@
     )
   )
-  (zone (net 45) (net_name "/RADIO-RX-PTT1") (layer "B.Cu") (hatch edge 0.508)
+  (zone (net 61) (net_name "/RADIO-PTT1") (layer "B.Cu") (hatch edge 0.508)
     (priority 10)
     (connect_pads (clearance 0.254))
@@
         (xy 123 110)
         (xy 117.5 110)
-        (xy 117.5 104.5)
-        (xy 123 104.5)
+        (xy 117.5 107.5)
+        (xy 123 107.5)
       )
     )
