File: kicad/k1-aioc/k1-aioc.kicad_sch (KiCad schematic)
At the start: 46 parts, among them J1 12401832E402A, J2 Conn_01x07_Male, Q1 BC847BS, U1 MIC5330-SSYML, U2 STM32F373CBTx, Y1 8MHz/20pF

Commit message: k1-aioc Rev 1.1 with PTT2 GPIO input capabilities
Parts:
- added R18, R19: 220R, Resistor_SMD:R_0603_1608Metric, symbol Device:R
Connections:
- net RADIO-RX-PTT1: now also R19.1
- net RADIO-VP-PTT2: now also R18.1
- net PTT1-IN: now reaches U2.42 (PB6)
- net PTT1-IN: now also R19.2
- net PTT2-IN: now reaches U2.43 (PB7)
- net PTT2-IN: now also R18.2
Other:
- note added: "GPIO Input (5V)"
- note added: "USART1-RX (5V)"
- note added: "USART1-TX (5V)"
- note removed: "USART1-RX"
- note removed: "USART1-TX"
- moved on the sheet: C11, C14, D1, D2, D3, D4, R16, R3, R5

Commit message: Changed PTT1 and RADIO-RX to a split-pad that is automatically connected, when a TRS connector is used. If not, then both pads can be used separately
Parts:
- R17: value N.M. -> 220R
Connections:
- net RADIO-RX-PTT1 renamed RADIO-PTT1
- net RADIO-PTT1: no longer R8.1
- net RADIO-VP-PTT2 renamed RADIO-PTT2
- new net RADIO-RX: R8.1
Other:
- note added: "K connector consists of two TRS connectors (3.5mm and 2.5mm) spaced 12mm apart Upper connector (2.5mm) T: SPK+ R: TxData (from Radio) S: GND Lower connector (3.5mm) T: +V/PTT2 R: MIC+ S: PTT1/RxData (to Radio) RADIO-RX and RADIO-PTT1 have a split-pad in the layout, which is automatically connected with each other, if a K1 connector layout is used."
- note removed: "K connector consists of two TRS connectors (3.5mm and 2.5mm) spaced 12mm apart Upper connector (2.5mm) T: SPK+ R: TxData (from Radio) S: GND Lower connector (3.5mm) T: +V/PTT2 R: MIC+ S: PTT1/RxData (to Radio)"
Changed lines of the file:
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@@
     (effects (font (size 1.27 1.27)) (justify left bottom))
   )
-  (text "K connector consists of two TRS connectors (3.5mm and 2.5mm) spaced 12mm apart\nUpper connector (2.5mm)\nT: SPK+\nR: TxData (from Radio)\nS: GND\n\nLower connector (3.5mm)\nT: +V/PTT2\nR: MIC+\nS: PTT1/RxData (to Radio)\n"
-    (at 166.37 39.37 0)
+  (text "K connector consists of two TRS connectors (3.5mm and 2.5mm) spaced 12mm apart\nUpper connector (2.5mm)\nT: SPK+\nR: TxData (from Radio)\nS: GND\n\nLower connector (3.5mm)\nT: +V/PTT2\nR: MIC+\nS: PTT1/RxData (to Radio)\n\nRADIO-RX and RADIO-PTT1 have a split-pad \nin the layout, which is automatically connected \nwith each other, if a K1 connector layout is used."
+    (at 163.83 41.91 0)
     (effects (font (size 1.27 1.27)) (justify left bottom))
   )
@@
     (effects (font (size 1.27 1.27)) (justify left bottom))
   )
-  (label "RADIO-VP-PTT2" (at 237.49 36.83 0)
+  (label "RADIO-PTT2" (at 237.49 36.83 0)
     (effects (font (size 1.27 1.27)) (justify left bottom))
   )
@@
     (effects (font (size 1.27 1.27)) (justify left bottom))
   )
-  (label "RADIO-RX-PTT1" (at 181.61 152.4 0)
+  (label "RADIO-PTT1" (at 181.61 152.4 0)
     (effects (font (size 1.27 1.27)) (justify left bottom))
   )
@@
     (effects (font (size 1.27 1.27)) (justify left bottom))
   )
-  (label "RADIO-VP-PTT2" (at 181.61 154.94 0)
+  (label "RADIO-PTT2" (at 181.61 154.94 0)
     (effects (font (size 1.27 1.27)) (justify left bottom))
   )
@@
     (effects (font (size 1.27 1.27)) (justify left bottom))
   )
-  (label "RADIO-RX-PTT1" (at 238.76 116.84 0)
+  (label "RADIO-RX" (at 238.76 116.84 0)
     (effects (font (size 1.27 1.27)) (justify left bottom))
   )
@@
     (effects (font (size 1.27 1.27)) (justify left bottom))
   )
-  (label "RADIO-RX-PTT1" (at 237.49 60.96 0)
+  (label "RADIO-PTT1" (at 237.49 60.96 0)
     (effects (font (size 1.27 1.27)) (justify left bottom))
   )
@@
     (in_bom yes) (on_board yes)
     (property "Reference" "R17" (id 0) (at 184.15 101.6 90))
-    (property "Value" "N.M." (id 1) (at 189.23 101.6 90))
+    (property "Value" "220R" (id 1) (at 189.23 101.6 90))
     (property "Footprint" "Resistor_SMD:R_0603_1608Metric" (id 2) (at 184.15 102.362 90)
       (effects (font (size 1.27 1.27)) hide)
@@
     )
     (path "/1d2bbe26-fe20-4f5c-9f43-026bf42bc8df"
-      (reference "R17") (unit 1) (value "N.M.") (footprint "Resistor_SMD:R_0603_1608Metric")
+      (reference "R17") (unit 1) (value "220R") (footprint "Resistor_SMD:R_0603_1608Metric")
     )
     (path "/6a7c960a-ea90-47ce-8d9a-a047368cb5f9"
